File: PCB/PowerRegulation/PowerRegulation.kicad_pcb (KiCad board)
At the start: 4 copper layers, 129 parts, among them J1 USB_C_Receptacle_USB2.0_14P, J3 Wii audio in, J4 OLED, SW1 RESET, SW2 BOOT, U1 BQ25883RGER, U10 MCP4651-503E/ST, U11 PAM8403, U2 TPS22918DBVR, U3 STM32F072CBTx, U4 TPS22918DBVR, U5 TPS563200DDCR, U6 TPS563200DDCR, U7 TPS563200DDCR, U8 TPS563200DDCR, U9 TPS563200DDCR

Commit message: made the aligment of the 1V, 1.15V, 1.8V and 3.3V regulators
Parts:
- moved C27 167.3 mm to (-48.7, 119.2)
- moved C29 167.3 mm to (-121.0, 177.5)
- moved C54 167.3 mm to (-108.8, 155.3)
- moved C55 167.3 mm to (-114.0, 152.0)
- moved C59 167.3 mm to (-110.5, 184.5)
- moved R15 167.3 mm to (-97.2, 145.4)
- moved C25 167.3 mm to (-53.4, 134.1)
- moved C26 167.3 mm to (-53.4, 137.1)
- moved C28 167.3 mm to (-58.4, 149.7)
- moved C30 167.3 mm to (-109.0, 139.5)
- moved C56 167.3 mm to (-111.0, 161.5)
- moved C57 167.3 mm to (-109.5, 168.0)
- moved C58 167.3 mm to (-110.5, 177.0)
- moved L5 167.3 mm to (-60.5, 185.2)
- moved R13 167.3 mm to (-103.0, 171.9)
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
Commit message: routed all voltage regulators
Parts:
- moved C29 290.7 mm to (161.0, 107.0), turned to -90 degrees
- moved C30 273.4 mm to (162.0, 103.5)
- moved C55 266.9 mm to (150.3, 115.0)
- moved C59 262.9 mm to (143.8, 118.0), turned to -90 degrees
- moved R13 257.5 mm to (146.5, 108.0), turned to -90 degrees
- moved C54 256.1 mm to (143.3, 110.0), turned to 90 degrees
- moved R15 255.6 mm to (156.0, 111.0)
- moved C57 234.7 mm to (119.0, 114.5)
- moved C58 230.8 mm to (112.5, 117.5), turned to -90 degrees
- moved L5 230.5 mm to (155.5, 104.5)
- moved C56 229.1 mm to (112.0, 109.0), turned to 90 degrees
- moved C28 214.1 mm to (151.7, 108.5), turned to 180 degrees
- moved U9 211.5 mm to (149.4, 104.1)
- moved U4 208.8 mm to (145.6, 114.0)
- moved C25 208.7 mm to (152.5, 99.5), turned to 90 degrees
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
Commit message: Layout the power circuit
Parts:
- added C60: 10uF, EasyEDA:R0805, F.Cu at (36.5, 87.0)
- added C61: 10uF, EasyEDA:R0805, F.Cu at (36.5, 103.5)
- added C62: 10uF, EasyEDA:R0805, F.Cu at (36.5, 95.0)
- moved TH1 152.7 mm to (76.5, 128.0)
- moved C49 126.0 mm to (211.4, 136.6)
- moved C39 123.1 mm to (83.5, 113.0)
- moved C40 123.1 mm to (81.5, 109.7)
- moved C41 123.1 mm to (91.0, 110.2)
- moved C42 123.1 mm to (91.0, 113.2)
- moved C43 123.1 mm to (81.5, 115.7)
- moved C44 123.1 mm to (90.5, 106.2)
- moved C53 123.1 mm to (79.0, 115.7)
- moved L6 123.1 mm to (86.0, 107.7)
- moved R22 123.1 mm to (90.5, 120.2)
- moved R23 123.1 mm to (86.0, 117.2)
- moved R24 123.1 mm to (93.0, 120.2)
- moved R25 123.1 mm to (86.0, 119.7)
- moved R27 123.1 mm to (93.5, 114.2)
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Other:
- board text added: "POWER"

Commit message: Add grounded screws
Parts:
- added C63: 10uF, EasyEDA:R0805, F.Cu at (69.2, 105.8)
- added C64: 10uF, EasyEDA:R0805, F.Cu at (69.8, 97.3)
- added H1: MountingHole_Pad, MountingHole:MountingHole_3.2mm_M3_Pad_Via, F.Cu at (66.4, 130.5)
- added H2: MountingHole_Pad, MountingHole:MountingHole_3.2mm_M3_Pad_Via, F.Cu at (186.2, 131.3)
- added H3: MountingHole_Pad, MountingHole:MountingHole_3.2mm_M3_Pad_Via, F.Cu at (106.0, 73.0)
- added H4: MountingHole_Pad, MountingHole:MountingHole_3.2mm_M3_Pad_Via, F.Cu at (186.5, 72.4)
- moved NT1 58.6 mm to (161.5, 107.0), turned to 90 degrees
- moved C1 35.7 mm to (79.8, 82.3)
- moved C10 35.7 mm to (98.8, 83.0)
- moved C11 35.7 mm to (97.2, 76.3)
- moved C12 35.7 mm to (93.2, 75.3)
- moved C13 35.7 mm to (79.8, 88.3)
- moved C14 35.7 mm to (77.8, 88.8)
- moved C15 35.7 mm to (75.8, 88.8)
- moved C16 35.7 mm to (79.5, 95.3)
- moved C17 35.7 mm to (86.2, 93.8)
- moved C18 35.7 mm to (87.2, 89.8)
- moved C19 35.7 mm to (96.8, 103.8)
- moved C2 35.7 mm to (86.8, 80.8)
- moved C20 35.7 mm to (99.2, 103.3)
- moved C21 35.7 mm to (101.2, 103.3)
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Connections:
- J4 pad 1: (no net) -> +3.3V
- J4 pad 2: (no net) -> GNDREF
- J4 pad 3: (no net) -> Net-(J4-SDA)
- J4 pad 4: (no net) -> Net-(J4-SCL)
- U3 pad 15: Net-(J4-Pin_3) -> Net-(J4-SDA)
- U3 pad 16: Net-(J4-Pin_4) -> Net-(J4-SCL)
Other:
- board outline added: 128 x 66.5 mm
- board text added: "3V3"
- board text added: "GND"
- board text added: "SCL"
- board text added: "SDA"
- board text removed: "OLED"
- board text removed: "POWER"

Commit message: make logo, route some stuff
THIS IS BEFORE THE BATT+ ON In2.Cu
Parts:
- J1: value USB_C_Receptacle_USB2.0_14P -> USB_C_Receptacle_USB2.0_16P; footprint EasyEDA:USB-C-SMD_TYPE-C-16PIN-2MD-073 -> Connector_USB:USB_C_Receptacle_Palconn_UTC16-G
- moved C44 24.3 mm to (112.0, 113.5), turned to 0 degrees
- moved R22 23.7 mm to (104.5, 120.5), turned to 180 degrees
- moved C39 23.4 mm to (100.5, 116.0), turned to 180 degrees
- moved R23 22.2 mm to (108.7, 122.8), turned to 90 degrees
- moved C40 22.2 mm to (99.8, 112.2)
- moved L6 22.2 mm to (104.2, 110.2)
- moved R24 22.2 mm to (111.2, 122.8)
- moved R25 22.2 mm to (104.2, 122.2)
- moved R27 22.2 mm to (111.8, 116.8)
- moved R28 22.2 mm to (109.8, 118.8)
- moved U1 22.2 mm to (105.2, 115.5)
- moved C42 22.0 mm to (109.2, 115.5)
- moved C41 21.4 mm to (108.0, 110.5), turned to -90 degrees
- moved TH1 18.1 mm to (95.5, 130.5)
- moved R32 15.7 mm to (162.0, 93.0), turned to -90 degrees
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Connections:
- net Net-(U3-PA11) renamed /Debug-
- net Net-(U3-PA12) renamed /Debug+
- J1 pad A8: (no net) -> unconnected-(J1-SBU1-PadA8)
- J1 pad B8: (no net) -> unconnected-(J1-SBU2-PadB8)
- U3 pad 46: unconnected-(U3-PB9-Pad46) -> CE
Routing:
- net VBUS: track 0.00 -> 112.1 mm
- net D-: track 0.00 -> 108.2 mm, vias 0 -> 2
- net D+: track 0.00 -> 104.4 mm, vias 0 -> 2
- net PG_BATT: track 0.00 -> 93.4 mm, vias 0 -> 4
- net INT_BATT: track 0.00 -> 71.4 mm, vias 0 -> 2
- net BATTERY+: track 0.00 -> 69.8 mm, vias 0 -> 10
- net SHDN: track 0.00 -> 69.5 mm, vias 0 -> 2
- net CE: track 0.00 -> 68.7 mm, vias 0 -> 4
- net Net-(LED1-C): track 0.00 -> 68.6 mm, vias 0 -> 2
- net MUTE: track 0.00 -> 66.6 mm, vias 0 -> 2
- net SDA_BATT: track 0.00 -> 65.2 mm, vias 0 -> 2
- net SCL_BATT: track 0.00 -> 58.3 mm, vias 0 -> 2
- net SCL_AUD: track 0.00 -> 47.9 mm
- net SDA_AUD: track 0.00 -> 47.5 mm, vias 0 -> 2
- net BOOT0: track 0.00 -> 45.6 mm
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Other:
- board size 128 x 66.5 mm -> 121.5 x 66.5 mm
- board text added: "DEBUG USB"
- board text added: "L"
- board text added: "Made by Matei, 15 RO"
- board text added: "PMS"
- board text added: "R"
- board text added: "v1"
- board text removed: "DEBUG"

Commit message: route the board
Parts:
- added TP12: TestPoint, TestPoint:TestPoint_Pad_D1.0mm, F.Cu at (146.0, 78.5)
- added TP13: TestPoint, TestPoint:TestPoint_Pad_D1.0mm, F.Cu at (90.0, 126.5)
- added TP14: L+, TestPoint:TestPoint_Pad_D2.5mm, F.Cu at (182.0, 103.0)
- added TP15: R+, TestPoint:TestPoint_Pad_D2.5mm, F.Cu at (182.0, 110.0)
- added TP16: GND, TestPoint:TestPoint_Pad_D2.5mm, F.Cu at (182.0, 117.0)
- added TP17: L-, TestPoint:TestPoint_Pad_D2.5mm, F.Cu at (182.0, 106.5)
- added TP18: R-, TestPoint:TestPoint_Pad_D2.5mm, F.Cu at (182.0, 113.5)
- added TP19: S, TestPoint:TestPoint_Pad_D2.0mm, F.Cu at (155.5, 133.5)
- added TP20: R, TestPoint:TestPoint_Pad_D2.0mm, F.Cu at (152.3, 133.5)
- added TP21: RN, TestPoint:TestPoint_Pad_D2.0mm, F.Cu at (149.3, 133.5)
- added TP22: T, TestPoint:TestPoint_Pad_D2.0mm, F.Cu at (146.3, 133.5)
- added TP23: TN, TestPoint:TestPoint_Pad_D2.0mm, F.Cu at (143.3, 133.5)
- moved R9 12.2 mm to (72.5, 92.5), turned to 180 degrees
- moved R12 11.5 mm to (104.5, 95.5), turned to 90 degrees
- moved R11 11.1 mm to (104.0, 99.5), turned to -90 degrees
- moved R15 10.1 mm to (80.5, 117.5), turned to 0 degrees
- moved R3 8.00 mm to (76.0, 85.0), turned to -90 degrees
- moved R13 6.63 mm to (75.5, 120.0), turned to 180 degrees
- moved R5 5.35 mm to (100.0, 85.0)
- moved R8 4.79 mm to (78.5, 97.5)
- moved C57 4.39 mm to (102.5, 87.5), turned to 90 degrees
- moved R4 3.91 mm to (98.5, 89.5)
- moved C62 3.26 mm to (66.0, 80.5), turned to 180 degrees
- moved R6 3.22 mm to (102.5, 82.5), turned to 0 degrees
- moved R1 2.77 mm to (72.5, 83.0)
- moved C10 2.56 mm to (98.0, 85.5)
- moved C56 2.18 mm to (107.5, 94.0)
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Routing:
- net +3.3V: track 8.94 -> 397.7 mm, vias 0 -> 20
- net PVDD: track 0.00 -> 179.0 mm, vias 0 -> 5
- net EN: track 0.00 -> 145.7 mm, vias 0 -> 5
- net +BATT: track 11.8 -> 125.1 mm, vias 0 -> 24
- net Net-(U2-QOD): track 0.00 -> 59.7 mm, vias 0 -> 2
- net GNDREF: track 0.00 -> 57.0 mm, vias 0 -> 126
- net 1.15V: track 0.00 -> 50.3 mm
- net AUDIOR: track 0.00 -> 45.4 mm
- net Net-(U4-QOD): track 0.00 -> 44.8 mm
- net +1V0: track 0.00 -> 43.9 mm, vias 0 -> 7
- net AUDIOL: track 0.00 -> 39.4 mm
- net +1V8: track 0.00 -> 39.3 mm, vias 0 -> 6
- net SPEAKER_L+: track 0.00 -> 38.1 mm, vias 0 -> 2
- net SPEAKER_L-: track 0.00 -> 34.2 mm, vias 0 -> 2
- net Net-(U10-P0W): track 0.00 -> 32.6 mm, vias 0 -> 2
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- added copper zone on In2.Cu, net +BATT
- added copper zone on B.Cu, net GNDA
- added copper zone on F.Cu, net GNDA
- added copper zone on B.Cu, net GNDREF
- added copper zone on F.Cu, net GNDREF
- added copper zone on In1.Cu, net GNDREF
Other:
- board text added: "Headphone Jack"
- board text added: "SPEAKER"

Commit message: fix some connections
Routing:
- net +BATT: track 125.1 -> 131.9 mm, vias 24 -> 26
- net GNDREF: track 57.0 -> 62.1 mm, vias 126 -> 129
Changed lines of the file:
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@@
+	)
+	(via
+		(at 107 80)
+		(size 0.6)
+		(drill 0.3)
+		(layers "F.Cu" "B.Cu")
+		(free yes)
+		(net "+BATT")
 	)
 	(via
@@
 	)
 	(via
+		(at 109 86)
+		(size 0.6)
+		(drill 0.3)
+		(layers "F.Cu" "B.Cu")
+		(free yes)
+		(net "+BATT")
+	)
+	(via
 		(at 73.75 110.25)
 		(size 0.8)
@@
 		(drill 0.4)
 		(layers "F.Cu" "B.Cu")
+		(net "+BATT")
+	)
+	(segment
+		(start 107 84)
+		(end 109 86)
+		(width 1.5)
+		(layer "B.Cu")
+		(net "+BATT")
+	)
+	(segment
+		(start 107 80)
+		(end 107 84)
+		(width 1.5)
+		(layer "B.Cu")
 		(net "+BATT")
 	)
@@
 		(end 150 84)
 		(width 0.25)
+		(layer "F.Cu")
+		(net "GNDREF")
+	)
+	(segment
+		(start 171.74 75.385)
+		(end 172.32 74.805)
+		(width 0.5)
 		(layer "F.Cu")
 		(net "GNDREF")
@@
 	)
 	(segment
+		(start 164.26 75.385)
+		(end 163.68 74.805)
+		(width 0.5)
+		(layer "F.Cu")
+		(net "GNDREF")
+	)
+	(segment
 		(start 96.75 85)
 		(end 97.029034 84.720966)
@@
 	)
 	(segment
+		(start 171.2 75.385)
+		(end 171.74 75.385)
+		(width 0.5)
+		(layer "F.Cu")
+		(net "GNDREF")
+	)
+	(segment
 		(start 156.429339 120.060661)
 		(end 157.060661 120.060661)
@@
 	)
 	(segment
+		(start 164.3675 79.5)
+		(end 164.08 79.2125)
+		(width 1)
+		(layer "F.Cu")
+		(net "GNDREF")
+	)
+	(segment
 		(start 171.05 117.63)
 		(end 171.13 117.63)
@@
 	)
 	(segment
+		(start 164.8 75.385)
+		(end 164.26 75.385)
+		(width 0.5)
+		(layer "F.Cu")
+		(net "GNDREF")
+	)
+	(segment
 		(start 106.01 116.25)
 		(end 105.26 115.5)
@@
 	)
 	(segment
+		(start 168.8675 79)
+		(end 169.58 79.7125)
+		(width 1)
+		(layer "F.Cu")
+		(net "GNDREF")
+	)
+	(segment
 		(start 171.13 117.63)
 		(end 173 119.5)
@@
 	)
 	(segment
+		(start 168.5 79)
+		(end 168.8675 79)
+		(width 1)
+		(layer "F.Cu")
+		(net "GNDREF")
+	)
+	(segment
 		(start 167.2 132.5)
 		(end 166 131.3)
@@
 	)
 	(segment
+		(start 165 79.5)
+		(end 164.3675 79.5)
+		(width 1)
+		(layer "F.Cu")
+		(net "GNDREF")
+	)
+	(segment
 		(start 161.75 125.25)
 		(end 161 126)
@@
 	)
 	(via
+		(at 157.5 98)
+		(size 0.6)
+		(drill 0.3)
+		(layers "F.Cu" "B.Cu")
+		(free yes)
+		(net "GNDREF")
+	)
+	(via
+		(at 165 79.5)
+		(size 0.6)
+		(drill 0.3)
+		(layers "F.Cu" "B.Cu")
+		(free yes)
+		(net "GNDREF")
+	)
+	(via
 		(at 91.5 70)
 		(size 0.6)
@@
 		(net "GNDREF")
 	)
+	(via
+		(at 168.5 79)
+		(size 0.6)
+		(drill 0.3)
+		(layers "F.Cu" "B.Cu")
+		(free yes)
+		(net "GNDREF")
+	)

Commit message: Finish the board
Parts:
- moved C10 0.50 mm to (98.5, 85.5)
- moved C43 0.50 mm to (110.0, 110.5)
- moved C53 0.50 mm to (112.5, 110.5)
- moved R15 0.50 mm to (80.5, 118.0)
- moved R25 0.50 mm to (104.2, 122.8)
- moved L5 0.30 mm to (78.2, 108.5)
- moved C41 0.25 mm to (108.3, 110.5)
- moved C52 0.13 mm to (173.0, 123.5)
Routing:
- net GNDREF: track 62.1 -> 69.4 mm, vias 129 -> 155
- net +3.3V: track 397.7 -> 392.7 mm, vias 20 -> 19
- net GNDA: track 11.5 -> 8.31 mm
- net +BATT: track 131.9 -> 133.2 mm
- net PG_BATT: track 93.4 -> 92.7 mm
- net SDA_BATT: track 65.2 -> 65.9 mm
Other:
- board text added: "Prototype 1"
