File: PCB/PowerRegulation/PowerRegulation.kicad_pcb (KiCad board)
At the start: 4 copper layers, 121.5 x 66.5 mm, 150 parts, among them J1 USB_C_Receptacle_USB2.0_16P, J3 Wii audio in, J4 OLED, SW1 RESET, SW2 BOOT, U1 BQ25883RGER, U10 MCP4651-503E/ST, U11 PAM8403, U2 TPS22918DBVR, U3 STM32F072CBTx, U4 TPS22918DBVR, U5 TPS563200DDCR, U6 TPS563200DDCR, U7 TPS563200DDCR, U8 TPS563200DDCR, U9 TPS563200DDCR

Commit message: Fix some minor layout issues
Parts:
- moved TP1 1.50 mm to (169.5, 96.5)
- moved TP2 1.50 mm to (165.0, 96.5)
- moved TP3 1.50 mm to (173.6, 96.5)
Routing:
- net /Debug-: track 36.2 -> 37.8 mm
Changed lines of the file:
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@@
 		(capping no)
 		(filling no)
-		(zone_defaults)
 		(pcbplotparams
 			(layerselection 0x00000000_00000000_55555555_5755f5ff)
@@
 	(footprint "TestPoint:TestPoint_Pad_D2.0mm"
 		(layer "F.Cu")
-		(at 168 96.5)
+		(at 169.5 96.5)
 		(descr "SMD pad as test Point, diameter 2.0mm")
 		(tags "test point SMD pad")
@@
 	(footprint "TestPoint:TestPoint_Pad_D2.0mm"
 		(layer "F.Cu")
-		(at 172.1 96.5)
+		(at 173.6 96.5)
 		(descr "SMD pad as test Point, diameter 2.0mm")
 		(tags "test point SMD pad")
@@
 	(footprint "TestPoint:TestPoint_Pad_D2.0mm"
 		(layer "F.Cu")
-		(at 163.5 96.5)
+		(at 165 96.5)
 		(descr "SMD pad as test Point, diameter 2.0mm")
 		(tags "test point SMD pad")
 		(property "Reference" "TP2"
-			(at 1 -2 0)
+			(at 0 -2 0)
 			(layer "F.SilkS")
 			(effects
@@
 	)
 	(gr_text "DEBUG USB"
-		(at 163.5 93 0)
+		(at 165 93 0)
 		(layer "F.SilkS")
 		(effects
@@
 	)
 	(segment
-		(start 151.125 79.556802)
-		(end 153.012023 77.669779)
+		(start 151.1 85.98)
+		(end 151.1 85.23)
 		(width 0.2)
 		(layer "F.Cu")
@@
 	)
 	(segment
-		(start 164.75 87.83)
-		(end 165.975001 87.83)
+		(start 167.475001 94.475001)
+		(end 169.5 96.5)
 		(width 0.2)
 		(layer "F.Cu")
@@
 	)
 	(segment
-		(start 151.125 85.205)
-		(end 151.125 79.556802)
+		(start 153.012023 77.669779)
+		(end 158.487977 77.669779)
 		(width 0.2)
 		(layer "F.Cu")
@@
 	)
 	(segment
-		(start 151.1 85.98)
-		(end 151.1 85.23)
+		(start 167.79998 85.443612)
+		(end 167.79998 88.016388)
+		(width 0.2)
+		(layer "F.Cu")
+		(net "/Debug+")
+	)
+	(segment
+		(start 158.487977 77.669779)
+		(end 165.998218 85.18002)
 		(width 0.2)
 		(layer "F.Cu")
@@
 	)
 	(segment
-		(start 157.987977 77.669779)
-		(end 165.948198 85.63)
+		(start 151.1 85.23)
+		(end 151.125 85.205)
 		(width 0.2)
 		(layer "F.Cu")
@@
 	)
 	(segment
-		(start 165.975001 94.475001)
-		(end 168 96.5)
+		(start 151.125 85.205)
+		(end 151.125 79.556802)
 		(width 0.2)
 		(layer "F.Cu")
@@
 	)
 	(segment
-		(start 165.975001 87.83)
-		(end 165.975001 94.475001)
+		(start 151.125 79.556802)
+		(end 153.012023 77.669779)
 		(width 0.2)
 		(layer "F.Cu")
@@
 	)
 	(segment
-		(start 151.1 85.23)
-		(end 151.125 85.205)
+		(start 165.998218 85.18002)
+		(end 167.536388 85.18002)
 		(width 0.2)
 		(layer "F.Cu")
@@
 	)
 	(segment
-		(start 153.012023 77.669779)
-		(end 157.987977 77.669779)
+		(start 167.475001 88.341367)
+		(end 167.475001 94.475001)
 		(width 0.2)
 		(layer "F.Cu")
@@
 	)
 	(segment
-		(start 164.75 85.63)
-		(end 164.75 87.83)
+		(start 167.536388 85.18002)
+		(end 167.79998 85.443612)
 		(width 0.2)
 		(layer "F.Cu")
@@
 	)
 	(segment
-		(start 165.948198 85.63)
-		(end 164.75 85.63)
+		(start 167.79998 88.016388)
+		(end 167.475001 88.341367)
 		(width 0.2)
 		(layer "F.Cu")
@@
 	)
 	(segment
-		(start 153.198419 78.119779)
-		(end 157.801581 78.119779)
+		(start 167.35 85.63)
+		(end 167.35 87.83)
 		(width 0.2)
 		(layer "F.Cu")
@@
 	)
 	(segment
-		(start 164.563612 85.18002)
-		(end 164.30002 85.443612)
+		(start 151.575 79.743198)
+		(end 153.198419 78.119779)
 		(width 0.2)
 		(layer "F.Cu")
@@
 	)
 	(segment
-		(start 164.861822 85.18002)
-		(end 164.563612 85.18002)
+		(start 167.35 87.83)
+		(end 167.024999 87.83)
 		(width 0.2)
 		(layer "F.Cu")
@@
 	)
 	(segment
-		(start 151.575 85.205)
-		(end 151.575 79.743198)
+		(start 151.6 85.23)
+		(end 151.575 85.205)
 		(width 0.2)
 		(layer "F.Cu")
@@
 	)
 	(segment
-		(start 164.30002 88.016388)
-		(end 165.524999 89.241367)
+		(start 158.301581 78.119779)
+		(end 165.811802 85.63)
 		(width 0.2)
 		(layer "F.Cu")
@@
 	)
 	(segment
-		(start 151.6 85.98)
-		(end 151.6 85.23)
+		(start 165.811802 85.63)
+		(end 167.35 85.63)
 		(width 0.2)
 		(layer "F.Cu")
@@
 	)
 	(segment
-		(start 151.575 79.743198)
-		(end 153.198419 78.119779)
-		(width 0.2)
-		(layer "F.Cu")
-		(net "/Debug-")
-	)
-	(segment
-		(start 151.6 85.23)
-		(end 151.575 85.205)
+		(start 151.6 85.98)
+		(end 151.6 85.23)
 		(width 0.2)
 		(layer "F.Cu")
@@
 	)
 	(segment
-		(start 164.30002 85.443612)
-		(end 164.30002 88.016388)
+		(start 167.024999 94.475001)
+		(end 165 96.5)
 		(width 0.2)
 		(layer "F.Cu")
@@
 	)
 	(segment
-		(start 165.524999 89.241367)
-		(end 165.524999 94.475001)
+		(start 167.024999 87.83)
+		(end 167.024999 94.475001)
 		(width 0.2)
 		(layer "F.Cu")
@@
 	)
 	(segment
-		(start 165.524999 94.475001)
-		(end 163.5 96.5)
+		(start 151.575 85.205)
+		(end 151.575 79.743198)
 		(width 0.2)
 		(layer "F.Cu")
@@
 	)
 	(segment
-		(start 157.801581 78.119779)
-		(end 164.861822 85.18002)
+		(start 153.198419 78.119779)
+		(end 158.301581 78.119779)
 		(width 0.2)
 		(layer "F.Cu")
